Commit message: updated motors

File: body.urdf (robot description, URDF)
Before this commit: robot robot, 3 links, 2 joints
Joints:
- joint Torso_BackLeg: origin xyz=0 -0.5 1 rpy=0 0 0 -> xyz=0.5 0 1 rpy=0 0 0
- joint Torso_FrontLeg: origin xyz=0 0.5 1 rpy=0 0 0 -> xyz=-0.5 0 1 rpy=0 0 0

Commit message: quadruped but legs in wrong places

File: body.urdf (robot description, URDF)
Before this commit: robot robot, 3 links, 2 joints
Links:
- added link LeftLeg, mass 1; collision box size=1 0.2 0.2; visual box size=1 0.2 0.2
- added link LowerBackLeg, mass 1; collision box size=0.2 0.2 1; visual box size=0.2 0.2 1
- added link LowerFrontLeg, mass 1; collision box size=0.2 0.2 1; visual box size=0.2 0.2 1
- added link LowerLeftLeg, mass 1; collision box size=0.2 0.2 1; visual box size=0.2 0.2 1
- added link LowerRightLeg, mass 1; collision box size=0.2 0.2 1; visual box size=0.2 0.2 1
- added link RightLeg, mass 1; collision box size=1 0.2 0.2; visual box size=1 0.2 0.2
- link BackLeg: geometry collision box size=0.2 1 0.2; visual box size=0.2 1 0.2
- link FrontLeg: geometry collision box size=0.2 1 0.2; visual box size=0.2 1 0.2
Joints:
- added joint BackLeg_LowerBackLeg: type revolute, parent BackLeg, child LowerBackLeg, origin xyz=0   - rpy=0 0 0, axis 1 0 0, limit lower=-3.14159 upper=3.14159 effort=0.0 velocity=0.0
- added joint FrontLeg_LowerFrontLeg: type revolute, parent FrontLeg, child LowerFrontLeg, origin xyz=0   1 rpy=0 0 0, axis 1 0 0, limit lower=-3.14159 upper=3.14159 effort=0.0 velocity=0.0
- added joint LeftLeg_LowerLeftLeg: type revolute, parent LeftLeg, child LowerLeftLeg, origin xyz=- 1   rpy=0 0 0, axis 0 1 0, limit lower=-3.14159 upper=3.14159 effort=0.0 velocity=0.0
- added joint RightLeg_LowerRightLeg: type revolute, parent RightLeg, child LowerRightLeg, origin xyz=1   0 rpy=0 0 0, axis 0 1 0, limit lower=-3.14159 upper=3.14159 effort=0.0 velocity=0.0
- added joint Torso_LeftLeg: type revolute, parent Torso, child LeftLeg, origin xyz=- 0 . rpy=0 0 0, axis 0 1 0, limit lower=-3.14159 upper=3.14159 effort=0.0 velocity=0.0
- added joint Torso_RightLeg: type revolute, parent Torso, child RightLeg, origin xyz=0 . 5 rpy=0 0 0, axis 0 1 0, limit lower=-3.14159 upper=3.14159 effort=0.0 velocity=0.0
- joint Torso_BackLeg: axis 0 1 0 -> 1 0 0; origin xyz=0.5 0 1 rpy=0 0 0 -> xyz=0   - rpy=0 0 0
- joint Torso_FrontLeg: axis 0 1 0 -> 1 0 0; origin xyz=-0.5 0 1 rpy=0 0 0 -> xyz=0   0 rpy=0 0 0

Commit message: switched out base code, readme research updates

File: body.urdf (robot description, URDF)
Before this commit: robot robot, 9 links, 8 joints
Joints:
- joint BackLeg_LowerBackLeg: origin xyz=0   - rpy=0 0 0 -> xyz=0 -1 0 rpy=0 0 0
- joint FrontLeg_LowerFrontLeg: origin xyz=0   1 rpy=0 0 0 -> xyz=0 1 0 rpy=0 0 0
- joint LeftLeg_LowerLeftLeg: origin xyz=- 1   rpy=0 0 0 -> xyz=-1 0 0 rpy=0 0 0
- joint RightLeg_LowerRightLeg: origin xyz=1   0 rpy=0 0 0 -> xyz=1 0 0 rpy=0 0 0
- joint Torso_BackLeg: origin xyz=0   - rpy=0 0 0 -> xyz=0 -0.5 1 rpy=0 0 0
- joint Torso_FrontLeg: origin xyz=0   0 rpy=0 0 0 -> xyz=0 0.5 1 rpy=0 0 0
- joint Torso_LeftLeg: origin xyz=- 0 . rpy=0 0 0 -> xyz=-0.5 0 1 rpy=0 0 0
- joint Torso_RightLeg: origin xyz=0 . 5 rpy=0 0 0 -> xyz=0.5 0 1 rpy=0 0 0

Commit message: hexapod basis
changes to generate body and brain toimplement 2 whoel new limbs

File: body.urdf (robot description, URDF)
Before this commit: robot robot, 9 links, 8 joints
Links:
- added link LowerFrontLeftLeg, mass 1; collision box size=0.2 0.2 1; visual box size=0.2 0.2 1
- added link LowerFrontRightLeg, mass 1; collision box size=0.2 0.2 1; visual box size=0.2 0.2 1
- added link frontLeftLeg, mass 1; collision box size=0.2 1 0.2; visual box size=0.2 1 0.2
- added link frontRightLeg, mass 1; collision box size=0.2 1 0.2; visual box size=0.2 1 0.2
Joints:
- added joint FrontLeftLeg_LowerFrontLeftLeg: type revolute, parent FrontLeftLeg, child LowerFrontLeftLeg, origin xyz=0 1 0 rpy=0 0 0, axis 1 0 0, limit lower=-3.14159 upper=3.14159 effort=0.0 velocity=0.0
- added joint FrontRightLeg_LowerFrontRightLeg: type revolute, parent FrontRightLeg, child LowerFrontRightLeg, origin xyz=0 1 0 rpy=0 0 0, axis 1 0 0, limit lower=-3.14159 upper=3.14159 effort=0.0 velocity=0.0
- added joint Torso_FrontLeftLeg: type revolute, parent Torso, child FrontLeftLeg, origin xyz=0 0.5 1 rpy=0 0 0, axis 1 0 0, limit lower=-3.14159 upper=3.14159 effort=0.0 velocity=0.0
- added joint Torso_FrontRightLeg: type revolute, parent Torso, child FrontRightLeg, origin xyz=0 0.5 1 rpy=0 0 0, axis 1 0 0, limit lower=-3.14159 upper=3.14159 effort=0.0 velocity=0.0

Commit message: implemented spheres

File: body.urdf (robot description, URDF)
Before this commit: robot robot, 13 links, 12 joints
Links:
- removed link LowerFrontLeftLeg
- removed link LowerFrontRightLeg
- removed link frontLeftLeg
- removed link frontRightLeg
- link Torso: geometry collision sphere radius=0.5; visual sphere radius=0.5
Joints:
- removed joint FrontLeftLeg_LowerFrontLeftLeg
- removed joint FrontRightLeg_LowerFrontRightLeg
- removed joint Torso_FrontLeftLeg
- removed joint Torso_FrontRightLeg

Commit message: moduar legs

File: body.urdf (robot description, URDF)
Before this commit: robot robot, 9 links, 8 joints
Links:
- removed link BackLeg
- removed link FrontLeg
- removed link LeftLeg
- removed link LowerBackLeg
- removed link LowerFrontLeg
- removed link LowerLeftLeg
- removed link LowerRightLeg
- removed link RightLeg
- added link LowerLeg0, mass 1; collision box size=0.2 0.2 1; visual box size=0.2 0.2 1
- added link LowerLeg1, mass 1; collision box size=0.2 0.2 1; visual box size=0.2 0.2 1
- added link LowerLeg2, mass 1; collision box size=0.2 0.2 1; visual box size=0.2 0.2 1
- added link LowerLeg3, mass 1; collision box size=0.2 0.2 1; visual box size=0.2 0.2 1
- added link LowerLeg4, mass 1; collision box size=0.2 0.2 1; visual box size=0.2 0.2 1
- added link LowerLeg5, mass 1; collision box size=0.2 0.2 1; visual box size=0.2 0.2 1
- added link LowerLeg6, mass 1; collision box size=0.2 0.2 1; visual box size=0.2 0.2 1
- added link LowerLeg7, mass 1; collision box size=0.2 0.2 1; visual box size=0.2 0.2 1
- added link UpperLeg0, mass 1; collision box size=1 0.2 0.2; visual box size=1 0.2 0.2
- added link UpperLeg1, mass 1; collision box size=1 0.2 0.2; visual box size=1 0.2 0.2
- added link UpperLeg2, mass 1; collision box size=1 0.2 0.2; visual box size=1 0.2 0.2
- added link UpperLeg3, mass 1; collision box size=1 0.2 0.2; visual box size=1 0.2 0.2
- added link UpperLeg4, mass 1; collision box size=1 0.2 0.2; visual box size=1 0.2 0.2
- added link UpperLeg5, mass 1; collision box size=1 0.2 0.2; visual box size=1 0.2 0.2
- added link UpperLeg6, mass 1; collision box size=1 0.2 0.2; visual box size=1 0.2 0.2
- added link UpperLeg7, mass 1; collision box size=1 0.2 0.2; visual box size=1 0.2 0.2
Joints:
- removed joint BackLeg_LowerBackLeg
- removed joint FrontLeg_LowerFrontLeg
- removed joint LeftLeg_LowerLeftLeg
- removed joint RightLeg_LowerRightLeg
- removed joint Torso_BackLeg
- removed joint Torso_FrontLeg
- removed joint Torso_LeftLeg
- removed joint Torso_RightLeg
- added joint Torso_UpperLeg0: type revolute, parent Torso, child UpperLeg0, origin xyz=0.5 0.0 1 rpy=0 0 0, axis 0.0 1.0 0, limit lower=-3.14159 upper=3.14159 effort=0.0 velocity=0.0
- added joint Torso_UpperLeg1: type revolute, parent Torso, child UpperLeg1, origin xyz=0.3535533905932738 0.3535533905932738 1 rpy=0 0 0, axis 0.7071067811865476 0.7071067811865476 0, limit lower=-3.14159 upper=3.14159 effort=0.0 velocity=0.0
- added joint Torso_UpperLeg2: type revolute, parent Torso, child UpperLeg2, origin xyz=3.061616997868383e-17 0.5 1 rpy=0 0 0, axis 1.0 6.123233995736766e-17 0, limit lower=-3.14159 upper=3.14159 effort=0.0 velocity=0.0
- added joint Torso_UpperLeg3: type revolute, parent Torso, child UpperLeg3, origin xyz=-0.35355339059327373 0.3535533905932738 1 rpy=0 0 0, axis 0.7071067811865476 0.7071067811865475 0, limit lower=-3.14159 upper=3.14159 effort=0.0 velocity=0.0
- added joint Torso_UpperLeg4: type revolute, parent Torso, child UpperLeg4, origin xyz=-0.5 6.123233995736766e-17 1 rpy=0 0 0, axis 1.2246467991473532e-16 1.0 0, limit lower=-3.14159 upper=3.14159 effort=0.0 velocity=0.0
- added joint Torso_UpperLeg5: type revolute, parent Torso, child UpperLeg5, origin xyz=-0.35355339059327384 -0.35355339059327373 1 rpy=0 0 0, axis 0.7071067811865475 0.7071067811865477 0, limit lower=-3.14159 upper=3.14159 effort=0.0 velocity=0.0
- added joint Torso_UpperLeg6: type revolute, parent Torso, child UpperLeg6, origin xyz=-9.184850993605148e-17 -0.5 1 rpy=0 0 0, axis 1.0 1.8369701987210297e-16 0, limit lower=-3.14159 upper=3.14159 effort=0.0 velocity=0.0
- added joint Torso_UpperLeg7: type revolute, parent Torso, child UpperLeg7, origin xyz=0.3535533905932737 -0.35355339059327384 1 rpy=0 0 0, axis 0.7071067811865477 0.7071067811865474 0, limit lower=-3.14159 upper=3.14159 effort=0.0 velocity=0.0
- added joint UpperLeg0_LowerLeg0: type revolute, parent UpperLeg0, child LowerLeg0, origin xyz=1.0 0.0 0 rpy=0 0 0, axis 0.0 1.0 0, limit lower=-3.14159 upper=3.14159 effort=0.0 velocity=0.0
- added joint UpperLeg1_LowerLeg1: type revolute, parent UpperLeg1, child LowerLeg1, origin xyz=0.7071067811865476 0.7071067811865476 0 rpy=0 0 0, axis 0.7071067811865476 0.7071067811865476 0, limit lower=-3.14159 upper=3.14159 effort=0.0 velocity=0.0
- added joint UpperLeg2_LowerLeg2: type revolute, parent UpperLeg2, child LowerLeg2, origin xyz=6.123233995736766e-17 1.0 0 rpy=0 0 0, axis 1.0 6.123233995736766e-17 0, limit lower=-3.14159 upper=3.14159 effort=0.0 velocity=0.0
- added joint UpperLeg3_LowerLeg3: type revolute, parent UpperLeg3, child LowerLeg3, origin xyz=-0.7071067811865475 0.7071067811865476 0 rpy=0 0 0, axis 0.7071067811865476 0.7071067811865475 0, limit lower=-3.14159 upper=3.14159 effort=0.0 velocity=0.0
- added joint UpperLeg4_LowerLeg4: type revolute, parent UpperLeg4, child LowerLeg4, origin xyz=-1.0 1.2246467991473532e-16 0 rpy=0 0 0, axis 1.2246467991473532e-16 1.0 0, limit lower=-3.14159 upper=3.14159 effort=0.0 velocity=0.0
- added joint UpperLeg5_LowerLeg5: type revolute, parent UpperLeg5, child LowerLeg5, origin xyz=-0.7071067811865477 -0.7071067811865475 0 rpy=0 0 0, axis 0.7071067811865475 0.7071067811865477 0, limit lower=-3.14159 upper=3.14159 effort=0.0 velocity=0.0
- added joint UpperLeg6_LowerLeg6: type revolute, parent UpperLeg6, child LowerLeg6, origin xyz=-1.8369701987210297e-16 -1.0 0 rpy=0 0 0, axis 1.0 1.8369701987210297e-16 0, limit lower=-3.14159 upper=3.14159 effort=0.0 velocity=0.0
- added joint UpperLeg7_LowerLeg7: type revolute, parent UpperLeg7, child LowerLeg7, origin xyz=0.7071067811865474 -0.7071067811865477 0 rpy=0 0 0, axis 0.7071067811865477 0.7071067811865474 0, limit lower=-3.14159 upper=3.14159 effort=0.0 velocity=0.0

Commit message: updated gifs

File: body.urdf (robot description, URDF)
Before this commit: robot robot, 17 links, 16 joints
Links:
- removed link LowerLeg4
- removed link LowerLeg5
- removed link LowerLeg6
- removed link LowerLeg7
- removed link UpperLeg4
- removed link UpperLeg5
- removed link UpperLeg6
- removed link UpperLeg7
Joints:
- removed joint Torso_UpperLeg4
- removed joint Torso_UpperLeg5
- removed joint Torso_UpperLeg6
- removed joint Torso_UpperLeg7
- removed joint UpperLeg4_LowerLeg4
- removed joint UpperLeg5_LowerLeg5
- removed joint UpperLeg6_LowerLeg6
- removed joint UpperLeg7_LowerLeg7
- joint Torso_UpperLeg1: axis 0.7071067811865476 0.7071067811865476 0 -> 1.0 6.123233995736766e-17 0; origin xyz=0.3535533905932738 0.3535533905932738 1 rpy=0 0 0 -> xyz=3.061616997868383e-17 0.5 1 rpy=0 0 0
- joint Torso_UpperLeg2: axis 1.0 6.123233995736766e-17 0 -> 1.2246467991473532e-16 1.0 0; origin xyz=3.061616997868383e-17 0.5 1 rpy=0 0 0 -> xyz=-0.5 6.123233995736766e-17 1 rpy=0 0 0
- joint Torso_UpperLeg3: axis 0.7071067811865476 0.7071067811865475 0 -> 1.0 1.8369701987210297e-16 0; origin xyz=-0.35355339059327373 0.3535533905932738 1 rpy=0 0 0 -> xyz=-9.184850993605148e-17 -0.5 1 rpy=0 0 0
- joint UpperLeg1_LowerLeg1: axis 0.7071067811865476 0.7071067811865476 0 -> 1.0 6.123233995736766e-17 0; origin xyz=0.7071067811865476 0.7071067811865476 0 rpy=0 0 0 -> xyz=6.123233995736766e-17 1.0 0 rpy=0 0 0
- joint UpperLeg2_LowerLeg2: axis 1.0 6.123233995736766e-17 0 -> 1.2246467991473532e-16 1.0 0; origin xyz=6.123233995736766e-17 1.0 0 rpy=0 0 0 -> xyz=-1.0 1.2246467991473532e-16 0 rpy=0 0 0
- joint UpperLeg3_LowerLeg3: axis 0.7071067811865476 0.7071067811865475 0 -> 1.0 1.8369701987210297e-16 0; origin xyz=-0.7071067811865475 0.7071067811865476 0 rpy=0 0 0 -> xyz=-1.8369701987210297e-16 -1.0 0 rpy=0 0 0
